File: BATAUS/BATAUS.kicad_pcb (KiCad board)
At the start: 2 copper layers, 13 parts, among them J1 TM1637, K1 SRA-05VDC-CL, Q1 MMBT2222A, U1 LM7805_TO220, U4 ESP32-C3_SUPERMINI_TH

Commit message: Alimentacion corregida
Parts:
- removed R1: R330, Resistor_THT:R_Axial_DIN0207_L6.3mm_D2.5mm_P10.16mm_Horizontal
- added R3: R10k, Resistor_THT:R_Axial_DIN0207_L6.3mm_D2.5mm_P10.16mm_Horizontal, F.Cu at (123.9, 76.0)
- J7: footprint TerminalBlock:TerminalBlock_Xinya_XY308-2.54-3P_1x03_P2.54mm_Horizontal -> TerminalBlock_4Ucon:TerminalBlock_4Ucon_1x03_P3.50mm_Vertical
- moved R2 26.3 mm to (120.0, 50.0), turned to -90 degrees
- moved Q1 4.04 mm to (97.0, 55.0), turned to -90 degrees
- moved J8 3.21 mm to (121.2, 85.3)
- moved U1 3.21 mm to (137.2, 71.0)
- moved C1 3.21 mm to (107.0, 75.5)
- moved D1 3.21 mm to (94.7, 59.0)
- moved J6 3.21 mm to (130.8, 85.3)
- moved J7 3.21 mm to (111.3, 85.3)
- moved K1 3.21 mm to (94.2, 71.4)
- moved R6 3.21 mm to (108.6, 79.8)
- moved U4 3.21 mm to (120.2, 64.5)
- moved J1 2.03 mm to (107.0, 57.1)
Connections:
- C1 pad 1: 5V -> 3.3V
- J6 pad 2: LvW2 -> 3.3V
- J7 pad 2: BP1 -> BP3
- J7 pad 3: GND -> BP1
- J8 pad 3: 5V -> 3.3V
- K1 pad NC: unconnected-(K1-PadNC) -> BP3
- R6 pad 1: 5V -> 3.3V
Routing:
- net 5V: track 146.2 -> 83.0 mm
- net 3.3V: track 46.1 -> 97.5 mm
- net BP3: track 0.00 -> 50.5 mm
- net Net-(Q1-B): track 6.39 -> 26.3 mm
- net LvW2: track 10.5 -> 0.00 mm
- net BP1: track 23.7 -> 16.3 mm
- net DatIN1: track 6.52 -> 8.67 mm
- net BP2: track 28.7 -> 27.3 mm
- net SCL: track 4.51 -> 5.59 mm
- net SDA: track 4.51 -> 5.59 mm
