File: BATAUS/BATAUS.kicad_sch (KiCad schematic)
At the start: 14 parts, among them J1 TM1637, K1 SRA-05VDC-CL, Q1 MMBT2222A, U1 LM7805_TO220, U4 ESP32-C3_SUPERMINI_TH

Commit message: Alimentacion corregida
Parts:
- removed R1: R330, Resistor_THT:R_Axial_DIN0207_L6.3mm_D2.5mm_P10.16mm_Horizontal, symbol Device:R
- J7: footprint TerminalBlock:TerminalBlock_Xinya_XY308-2.54-3P_1x03_P2.54mm_Horizontal -> TerminalBlock_4Ucon:TerminalBlock_4Ucon_1x03_P3.50mm_Vertical
Connections:
- net LvW2 is gone; now on net LvW: J6.3 (Pin_3)
- net 3.3V: now also J6.2 (Pin_2), J8.3 (Pin_3); no longer J8.2 (Pin_2)
- net BP1: now also J7.3 (Pin_3); no longer J7.2 (Pin_2)
- net GND: now also J8.2 (Pin_2); no longer J7.3 (Pin_3), J8.3 (Pin_3)
- net LvW: no longer J6.2 (Pin_2)
- net BP3: now reaches K1.NC
- net BP3: now also J7.2 (Pin_2)
